File: slow_precharge_latching_switch.sch (KiCad schematic (older format))
At the start: 22 parts

Commit message: saving it in this branch, gonna toss it soon
Parts:
- removed SW?: DPST_Switch, symbol DPST_Switch
- added P?: CONN_01X02, symbol CONN_01X02
- added R? (x2): 10K, symbol R
- added R?: 1K, symbol R
- added U?: TLP291, SOP-4, symbol TLP291
- R? (x2): value 100R -> 100
Connections:
- wire segments 70 -> 77
Other:
- moved on the sheet: Q?, R?
